Commit message: w

File: description/depth_camera.xacro (robot description, xacro)
@@ -5,5 +5,5 @@
         <parent link="chassis_link"/>
         <child link="camera_link"/>
-        <origin xyz="-0.05 0.26 -0.1" rpy="-1.570796 0 0"/>
+        <origin xyz="-0.05 0.26 -0" rpy="-1.570796 0 0"/>
     </joint>
     <!-- Camera Link -->

File: description/lidar.xacro (robot description, xacro)
@@ -1,16 +1,55 @@
 <?xml version="1.0"?>
 <robot xmlns:xacro="http://www.ros.org/wiki/xacro">
-    <!-- Fix Lidar Message type -->
-    <!-- Fix vertical sampling-->
-    <!-- Lidar Joint -->
-    <joint name="lidar_joint" type="fixed">
+    <!-- Lidar Base -->
+    <joint name="lidar_base_joint" type="fixed">
         <parent link="chassis_link"/>
-        <child link="lidar_link"/>
+        <child link="lidar_base_link"/>
         <origin xyz="0 0 -0.23" rpy="0 0 0"/>
     </joint>
-    <!-- Lidar Link -->
+    <link name="lidar_base_link">
+        <visual>
+            <origin xyz="-0.085 -0.2 -0.11" rpy="1.57 0 1.57"/>
+            <geometry>
+                <mesh filename="file:$(find kridtbot)/meshes/lidar_stand_base.STL" scale="0.001 0.001 0.001"/>
+            </geometry>
+            <material name="orange"/>
+        </visual>
+        <collision>
+            <origin xyz="-0.085 -0.2 -0.11" rpy="1.57 0 1.57"/>
+            <geometry>
+                <mesh filename="file:$(find kridtbot)/meshes/lidar_stand_base.STL" scale="0.001 0.001 0.001"/>
+            </geometry>
+        </collision>
+    </link>
+    <!-- Lidar Stand -->
+    <joint name="lidar_stand_joint" type="fixed">
+        <parent link="lidar_base_link"/>
+        <child link="lidar_stand_link"/>
+        <origin xyz="0 0 0" rpy="0 0 0"/>
+    </joint>
+    <link name="lidar_stand_link">
+        <visual>
+            <origin xyz="0.08 -0.2 0" rpy="-1.57 0 1.57"/>
+            <geometry>
+                <mesh filename="file:$(find kridtbot)/meshes/lidar_stand_top.STL" scale="0.001 0.001 0.001"/>
+            </geometry>
+            <material name="orange"/>
+        </visual>
+        <collision>
+            <origin xyz="0.08 -0.2 0" rpy="-1.57 0 1.57"/>
+            <geometry>
+                <mesh filename="file:$(find kridtbot)/meshes/lidar_stand_top.STL" scale="0.001 0.001 0.001"/>
+            </geometry>
+        </collision>
+    </link>
+    <!-- Lidar -->
+    <joint name="lidar_joint" type="fixed">
+        <parent link="lidar_stand_link"/>
+        <child link="lidar_link"/>
+        <origin xyz="-0.002 -0.135 -0.185" rpy="0 0 0"/>
+    </joint>
     <link name="lidar_link">
         <visual>
-            <origin xyz="0 0 0" rpy="-1.578 0 0"/>
+            <origin xyz="0 0 0" rpy="1.57 0 1.57"/>
             <geometry>
                 <mesh filename="file:$(find kridtbot)/meshes/mid-360-asm copy.STL" scale="0.001 0.001 0.001"/>
@@ -19,5 +58,5 @@
         </visual>
         <collision>
-            <origin xyz="0 0 0" rpy="-1.578 0 0"/>
+            <origin xyz="0 0 0" rpy="0 0 0"/>
             <geometry>
                 <mesh filename="file:$(find kridtbot)/meshes/mid-360-asm copy.STL" scale="0.001 0.001 0.001"/>
@@ -25,44 +64,35 @@
         </collision>
     </link>
-    <!-- FOV -->
-    <link name="lidar_optical_link">
-        <visual>
-            <geometry>
-                <mesh filename="file:$(find kridtbot)/meshes/mid-360-fov-asm.STL" scale="0.001 0.001 0.001"/>
-            </geometry>
-            <material name="blue opaque"/>
-        </visual>
-    </link>
-    <joint name="lidar_optical_joint" type="fixed">
-        <parent link="lidar_link"/>
-        <child link="lidar_optical_link"/>
-        <origin xyz="0 0 -0.02" rpy="-1.578 0 0"/>
-    </joint>
     <!-- Gazebo Sensor Definition -->
     <gazebo reference="lidar_link">
         <sensor type="gpu_lidar" name="lidar_sensor">
-            <visualize>false</visualize>  <!-- Visualization causes crashes, disable if needed -->
-            <pose>0 0 0 0 0 0</pose>
-            <update_rate>10</update_rate>  <!-- 10 Hz scan update -->
+            <visualize>true</visualize>
+            <pose>0 0 0 0 0 0</pose> <!-- 180 deg flip -->
+            <update_rate>100</update_rate>
             <lidar>
-            <!-- Information from Livox specs -->
                 <scan>
                     <horizontal>
-                        <samples>360</samples>  <!-- 360 points per rotation -->
-                        <!--<resolution>1</resolution> -->
-                        <min_angle>-3.14</min_angle>
-                        <max_angle>3.14</max_angle>
+                        <samples>360</samples>
+                        <resolution>1</resolution>
+                        <min_angle>0</min_angle>
+                        <max_angle>6.283185</max_angle> <!-- 360 deg -->
                     </horizontal>
                     <vertical>
-                        <samples>10</samples>  <!-- 1 vertical scan -->
-                        <min_angle>0</min_angle>
-                        <max_angle>-1</max_angle>
+                        <samples>100</samples>
+                        <resolution>1</resolution>
+                        <min_angle>-0.122</min_angle> <!-- -7.22 deg -->
+                        <max_angle>0.9</max_angle>  <!-- 55.22 deg seems to be to much-->
                     </vertical>
                 </scan>
                 <range>
-                    <min>0.1</min>  <!-- 10 cm min detection -->
-                    <max>12</max>  <!-- 70 m max detection -->
-                    <!--<resolution>0.02</resolution> -->  <!-- 2 cm precision -->
+                    <min>0.1</min>
+                    <max>200.0</max>
+                    <resolution>0.002</resolution>
                 </range>
+                <noise>
+                    <type>gaussian</type>
+                    <mean>0.0</mean>
+                    <stddev>0.01</stddev>
+                </noise>
             </lidar>
             <topic>lidar/points</topic>

File: description/robot_core.xacro (robot description, xacro)
@@ -155,9 +155,35 @@
     <material>Gazebo/Black</material>
   </gazebo>
+  <!-- _____________LEFT REAR motor ____________-->
+  <joint name="left_rear_motor" type="fixed">
+    <origin xyz="0.0012158 0 0.2449" rpy="1.5708 0 0"/>
+    <axis xyz="0 0 1"/>
+    <parent link="left_rear_lin_link"/>
+    <child link="left_rear_motor_link"/>
+  </joint>
+  <link name="left_rear_motor_link">
+    <visual>
+      <origin xyz="0 0 0.04675" rpy="0 0 0"/>
+      <geometry>
+        <cylinder radius="0.049" length="0.0395"/> <!-- From myactuator specifications-->
+      </geometry>
+      <material name="black"/>
+    </visual>
+    <collision>
+      <origin xyz="0 0 0" rpy="0 0 0"/>
+      <geometry>
+        <cylinder radius="0.049" length="0.0395"/>
+      </geometry>
+    </collision>
+    <inertial>
+      <mass value="1.01100"/>
+      <inertia ixx="5844491.97e-9" ixy="-376.28e-9" ixz="-3671.08e-9" iyy="5842839.83e-9" iyz="-796.72e-9" izz="3646247.90e-9"/>
+    </inertial>
+  </link>
   <!-- _____________LEFT REAR wheel ____________-->
   <joint name="left_rear_wheel" type="continuous">
-    <origin xyz="0.0012158 0 0.2449" rpy="1.5708 0 0"/>
-    <axis xyz="0 0 1"/>
-    <parent link="left_rear_lin_link"/>
+    <origin xyz="0 0 0" rpy="0 0 0"/>
+    <axis xyz="0 0 1"/>
+    <parent link="left_rear_motor_link"/>
     <child link="left_rear_rev_link"/>
     <dynamics damping="0.7" friction="1"/>
@@ -165,14 +191,15 @@
   <link name="left_rear_rev_link">
     <visual>
-      <origin xyz="0 0 0.06266" rpy="0 0 0"/>
-      <geometry>
-        <cylinder radius="0.0865" length="0.05234"/>
+      <origin xyz="-0.085 0.085 0.035" rpy="1.57 0 0"/>
+      <geometry>
+        <!--<cylinder radius="0.0865" length="0.05234"/>-->
+        <mesh filename="file:$(find kridtbot)/meshes/wheel_assem.STL" scale="0.001 0.001 0.001"/>
       </geometry>
       <material name="orange"/>
     </visual>
     <collision>
-      <origin xyz="0 0 0.06266" rpy="0 0 0"/>
-      <geometry>
-        <cylinder radius="0.0865" length="0.05234"/>
+      <origin xyz="-0.085 0.085 0.035" rpy="1.57 0 0"/>
+      <geometry>
+        <mesh filename="file:$(find kridtbot)/meshes/wheel_assem.STL" scale="0.001 0.001 0.001"/>
       </geometry>
       <material name="mesh_color"/>
@@ -221,9 +248,35 @@
     <material>Gazebo/Black</material>
   </gazebo>
+ <!-- _____________LEFT front motor ____________-->
+<joint name="left_front_motor" type="fixed">
+    <origin xyz="0.0012158 0 0.2449" rpy="1.5708 0 0"/>
+    <axis xyz="0 0 1"/>
+    <parent link="left_front_lin_link"/>
+    <child link="left_front_motor_link"/>
+  </joint>
+  <link name="left_front_motor_link">
+    <visual>
+      <origin xyz="0 -0.02 0.04675" rpy="0 0 0"/>
+      <geometry>
+        <cylinder radius="0.049" length="0.0395"/> <!-- From myactuator specifications-->
+      </geometry>
+      <material name="black"/>
+    </visual>
+    <collision>
+      <origin xyz="0 0 0" rpy="0 0 0"/>
+      <geometry>
+        <cylinder radius="0.049" length="0.0395"/>
+      </geometry>
+    </collision>
+    <inertial>
+      <mass value="1.01100"/>
+      <inertia ixx="5844491.97e-9" ixy="-376.28e-9" ixz="-3671.08e-9" iyy="5842839.83e-9" iyz="-796.72e-9" izz="3646247.90e-9"/>
+    </inertial>
+  </link>
   <!-- _____________LEFT FRONT wheel ____________-->
   <joint name="left_front_wheel" type="continuous">
-    <origin xyz="0.0012158 0 0.2449" rpy="1.5708 0 0"/>
-    <axis xyz="0 0 1"/>
-    <parent link="left_front_lin_link"/>
+    <origin xyz="0 0 0" rpy="0 0 0"/>
+    <axis xyz="0 0 1"/>
+    <parent link="left_front_motor_link"/>
     <child link="left_front_rev_link"/>
     <dynamics damping="0.7" friction="1"/>
@@ -231,14 +284,15 @@
   <link name="left_front_rev_link">
     <visual>
-      <origin xyz="0 0 0.06266" rpy="0 0 0"/>
-      <geometry>
-        <cylinder radius="0.0865" length="0.05234"/>
+      <origin xyz="-0.085 0.085 0.035" rpy="1.57 0 0"/>
+      <geometry>
+        <!--<cylinder radius="0.0865" length="0.05234"/>-->
+        <mesh filename="file:$(find kridtbot)/meshes/wheel_assem.STL" scale="0.001 0.001 0.001"/>
       </geometry>
       <material name="orange"/>
     </visual>
     <collision>
-      <origin xyz="0 0 0.06266" rpy="0 0 0"/>
-      <geometry>
-        <cylinder radius="0.0865" length="0.05234"/>
+      <origin xyz="-0.085 0.085 0.035" rpy="1.57 0 0"/>
+      <geometry>
+        <mesh filename="file:$(find kridtbot)/meshes/wheel_assem.STL" scale="0.001 0.001 0.001"/>
       </geometry>
       <material name="mesh_color"/>
@@ -250,5 +304,5 @@
   </link>
   <gazebo reference="left_front_rev_link">
-    <material>Gazebo/Black</material>
+    <material>Gazebo/Orange</material>
     <mu1 value="3"/>
     <mu2 value="3"/>
@@ -322,9 +376,35 @@
     <material>Gazebo/Black</material>
   </gazebo>
+   <!-- _____________Right REAR motor ____________-->
+  <joint name="right_rear_motor" type="fixed">
+    <origin xyz="0.0012158 0 0.2449" rpy="1.5708 0 0"/>
+    <axis xyz="0 0 1"/>
+    <parent link="right_rear_lin_link"/>
+    <child link="right_rear_motor_link"/>
+  </joint>
+  <link name="right_rear_motor_link">
+    <visual>
+      <origin xyz="0 0 0.04675" rpy="0 0 0"/>
+      <geometry>
+        <cylinder radius="0.049" length="0.0395"/> <!-- From myactuator specifications-->
+      </geometry>
+      <material name="black"/>
+    </visual>
+    <collision>
+      <origin xyz="0 0 0" rpy="0 0 0"/>
+      <geometry>
+        <cylinder radius="0.049" length="0.0395"/>
+      </geometry>
+    </collision>
+    <inertial>
+      <mass value="1.01100"/>
+      <inertia ixx="5844491.97e-9" ixy="-376.28e-9" ixz="-3671.08e-9" iyy="5842839.83e-9" iyz="-796.72e-9" izz="3646247.90e-9"/>
+    </inertial>
+  </link>
   <!-- _____________RIGHT REAR wheel ____________-->
   <joint name="right_rear_wheel" type="continuous">
-    <origin xyz="0.0012158 0 0.2449" rpy="1.5708 0 0"/>
-    <axis xyz="0 0 1"/>
-    <parent link="right_rear_lin_link"/>
+    <origin xyz="0 0 0" rpy="0 0 0"/>
+    <axis xyz="0 0 1"/>
+    <parent link="right_rear_motor_link"/>
     <child link="right_rear_rev_link"/>
     <dynamics damping="0.7" friction="1"/>
@@ -332,14 +412,15 @@
   <link name="right_rear_rev_link">
     <visual>
-      <origin xyz="0 0 0.06266" rpy="0 0 0"/>
-      <geometry>
-        <cylinder radius="0.0865" length="0.05234"/>
+       <origin xyz="-0.085 0.085 0.035" rpy="1.57 0 0"/>
+      <geometry>
+        <!-- <cylinder radius="0.0865" length="0.05234"/> -->
+        <mesh filename="file:$(find kridtbot)/meshes/wheel_assem.STL" scale="0.001 0.001 0.001"/>
       </geometry>
       <material name="orange"/>
     </visual>
     <collision>
-      <origin xyz="0 0 0.06266" rpy="0 0 0"/>
-      <geometry>
-        <cylinder radius="0.0865" length="0.05234"/>
+       <origin xyz="-0.085 0.085 0.035" rpy="1.57 0 0"/>
+      <geometry>
+        <mesh filename="file:$(find kridtbot)/meshes/wheel_assem.STL" scale="0.001 0.001 0.001"/>
       </geometry>
       <material name="mesh_color"/>
@@ -390,9 +471,35 @@
     <material>Gazebo/Black</material>
   </gazebo>
+    <!-- _____________Right front motor ____________-->
+  <joint name="right_front_motor" type="fixed">
+    <origin xyz="0.0012158 0 0.2449" rpy="1.5708 0 0"/>
+    <axis xyz="0 0 1"/>
+    <parent link="right_front_lin_link"/>
+    <child link="right_front_motor_link"/>
+  </joint>
+  <link name="right_front_motor_link">
+    <visual>
+      <origin xyz="0 0 0.04675" rpy="0 0 0"/>
+      <geometry>
+        <cylinder radius="0.049" length="0.0395"/> <!-- From myactuator specifications-->
+      </geometry>
+      <material name="black"/>
+    </visual>
+    <collision>
+      <origin xyz="0 0 0" rpy="0 0 0"/>
+      <geometry>
+        <cylinder radius="0.049" length="0.0395"/>
+      </geometry>
+    </collision>
+    <inertial>
+      <mass value="1.01100"/>
+      <inertia ixx="5844491.97e-9" ixy="-376.28e-9" ixz="-3671.08e-9" iyy="5842839.83e-9" iyz="-796.72e-9" izz="3646247.90e-9"/>
+    </inertial>
+  </link>
   <!-- _____________RIGHT FRONT wheel ____________-->
   <joint name="right_front_wheel" type="continuous">
-    <origin xyz="0.0012158 0 0.2449" rpy="1.5708 0 0"/>
-    <axis xyz="0 0 1"/>
-    <parent link="right_front_lin_link"/>
+    <origin xyz="0.0 0 0" rpy="0 0 0"/>
+    <axis xyz="0 0 1"/>
+    <parent link="right_front_motor_link"/>
     <child link="right_front_rev_link"/>
     <dynamics damping="0.7" friction="1"/>
@@ -400,14 +507,15 @@
   <link name="right_front_rev_link">
     <visual>
-      <origin xyz="0 0 0.06266" rpy="0 0 0"/>
-      <geometry>
-        <cylinder radius="0.0865" length="0.05234"/>
+      <origin xyz="-0.085 0.085 0.035" rpy="1.57 0 0"/>
+      <geometry>
+        <!-- <cylinder radius="0.0865" length="0.05234"/> -->
+        <mesh filename="file:$(find kridtbot)/meshes/wheel_assem.STL" scale="0.001 0.001 0.001"/>
       </geometry>
       <material name="orange"/>
     </visual>
     <collision>
-      <origin xyz="0 0 0.06266" rpy="0 0 0"/>
-      <geometry>
-        <cylinder radius="0.0865" length="0.05234"/>
+      <origin xyz="-0.085 0.085 0.035" rpy="1.57 0 0"/>
+      <geometry>
+        <mesh filename="file:$(find kridtbot)/meshes/wheel_assem.STL" scale="0.001 0.001 0.001"/>
       </geometry>
       <material name="mesh_color"/>
