Commit message: lastest_update

File: description/depth_camera.xacro (robot description, xacro)
@@ -30,5 +30,5 @@
     </link>
     <!-- Gazebo Sensor Definition -->
-    <gazebo reference="camera_link">
+   <!-- <gazebo reference="camera_link">
         <material>Gazebo/Black</material>
         <sensor name="camera" type="depth">
@@ -36,16 +36,16 @@
             <visualize>true</visualize>
             <pose> 0 0 0 0 -1.57 -1.57</pose>
-            <update_rate>30</update_rate>  <!-- fps-->
+            <update_rate>30</update_rate>
             <camera>
                 <camera_info_topic>camera/camera_info</camera_info_topic>
-                <horizontal_fov>1.43</horizontal_fov> <!--oak-d depth fov -->
+                <horizontal_fov>1.43</horizontal_fov>
                 <image>
-                    <format>R8G8B8</format> <!--Not used since depth -->
-                    <width>1280</width> <!--oak-d -->
-                    <height>800</height>   <!--oadk-d -->
+                    <format>R8G8B8</format>
+                    <width>1280</width>
+                    <height>800</height>
                 </image>
                 <clip>
                     <near>0.7</near>
-                    <far>12</far>  <!--oak-d ideal depth rangee-->
+                    <far>12</far>
                 </clip>
             </camera>
@@ -53,4 +53,4 @@
             <gz_frame_id>camera_optical_link</gz_frame_id>
         </sensor>
-    </gazebo>
+    </gazebo> -->
 </robot>

File: description/imu.xacro (robot description, xacro)
@@ -96,5 +96,12 @@
           </noise>
         </z>
+        <w>
+        <noise type="gaussian">
+          <mean>0.0</mean>
+          <stddev>2e-3</stddev>
+        </noise>
+      </w>
       </orientation>
+      <orientation_covariance>0.0001 0 0 0 0 0 0 0 0 0.0001 0 0 0 0 0.0001</orientation_covariance>
         </imu>
         </sensor>

File: description/lidar.xacro (robot description, xacro)
@@ -73,5 +73,5 @@
                 <scan>
                     <horizontal>
-                        <samples>360</samples>
+                        <samples>720</samples>
                         <resolution>1</resolution>
                         <min_angle>0</min_angle>
@@ -87,5 +87,5 @@
                 <range>
                     <min>0.1</min>
-                    <max>200.0</max>
+                    <max>70.0</max>
                     <resolution>0.002</resolution>
                 </range>
@@ -93,5 +93,5 @@
                     <type>gaussian</type>
                     <mean>0.0</mean>
-                    <stddev>0.01</stddev>
+                    <stddev>0.0001</stddev>
                 </noise>
             </lidar>

File: description/robot.urdf.xacro (robot description, xacro)
@@ -1,8 +1,16 @@
 <?xml version="1.0"?>
-<robot xmlns:xacro="http://www.ros.org/wiki/xacro"  name="robot">
+<robot xmlns:xacro="http://www.ros.org/wiki/xacro"  name="robot" xmlns:gz="http://gazebosim.org/schema">
     <!-- Arguments -->
     <xacro:arg name="use_sim_system" default="false"/>
+    <xacro:arg name="use_skid" default="true"/>
     <!-- URDF Robot Description-->
     <xacro:include filename="robot_core.xacro" />
+    <!-- wheels -->
+    <xacro:if value="$(arg use_skid)">
+        <xacro:include filename="wheels_skid.xacro" />
+    </xacro:if>
+    <xacro:unless value="$(arg use_skid)">
+        <xacro:include filename="wheels_mec.xacro" />
+    </xacro:unless>
     <!-- Sensors -->
     <xacro:include filename="lidar.xacro" />

File: description/robot_core.xacro (robot description, xacro)
@@ -1,4 +1,4 @@
 <?xml version="1.0"?>
-<robot xmlns:xacro="http://www.ros.org/wiki/xacro">
+<robot xmlns:xacro="http://www.ros.org/wiki/xacro" xmlns:gz="http://gazebosim.org/schema">
   <!-- Materials -->
   <material name="orange">
@@ -153,5 +153,5 @@
   </link>
   <gazebo reference="left_rear_lin_link">
-    <material>Gazebo/Black</material>
+    <material>Gazebo/Red</material>
   </gazebo>
   <!-- _____________LEFT REAR motor ____________-->
@@ -181,40 +181,4 @@
     </inertial>
   </link>
-  <!-- _____________LEFT REAR wheel ____________-->
-  <joint name="left_rear_wheel" type="continuous">
-    <origin xyz="0 0 0" rpy="0 0 0"/>
-    <axis xyz="0 0 1"/>
-    <parent link="left_rear_motor_link"/>
-    <child link="left_rear_rev_link"/>
-    <dynamics damping="0.7" friction="1"/>
-  </joint>
-  <link name="left_rear_rev_link">
-    <visual>
-      <origin xyz="-0.085 0.085 0.035" rpy="1.57 0 0"/>
-      <geometry>
-        <!--<cylinder radius="0.0865" length="0.05234"/>-->
-        <mesh filename="file:$(find kridtbot)/meshes/wheel_assem.STL" scale="0.001 0.001 0.001"/>
-      </geometry>
-      <material name="orange"/>
-    </visual>
-    <collision>
-      <origin xyz="-0.085 0.085 0.035" rpy="1.57 0 0"/>
-      <geometry>
-        <mesh filename="file:$(find kridtbot)/meshes/wheel_assem.STL" scale="0.001 0.001 0.001"/>
-      </geometry>
-      <material name="mesh_color"/>
-    </collision>
-    <inertial>
-      <mass value="1.01100"/>
-      <inertia ixx="5844491.97e-9" ixy="-376.28e-9" ixz="-3671.08e-9" iyy="5842839.83e-9" iyz="-796.72e-9" izz="3646247.90e-9"/>
-    </inertial>
-  </link>
-  <gazebo reference="left_rear_rev_link">
-    <material>Gazebo/Orange</material>
-    <mu1 value="3"/>
-    <mu2 value="3"/>
-    <kp>1000000.0</kp>
-    <kd>1.0</kd>
-  </gazebo>
   <!-- _____________LEFT FRONT LINEAR actuator____________-->
   <joint name="left_front_linear" type="prismatic">
@@ -246,5 +210,5 @@
   </link>
   <gazebo reference="left_front_lin_link">
-    <material>Gazebo/Black</material>
+    <material>Gazebo/Red</material>
   </gazebo>
  <!-- _____________LEFT front motor ____________-->
@@ -274,42 +238,4 @@
     </inertial>
   </link>
-  <!-- _____________LEFT FRONT wheel ____________-->
-  <joint name="left_front_wheel" type="continuous">
-    <origin xyz="0 0 0" rpy="0 0 0"/>
-    <axis xyz="0 0 1"/>
-    <parent link="left_front_motor_link"/>
-    <child link="left_front_rev_link"/>
-    <dynamics damping="0.7" friction="1"/>
-  </joint>
-  <link name="left_front_rev_link">
-    <visual>
-      <origin xyz="-0.085 0.085 0.035" rpy="1.57 0 0"/>
-      <geometry>
-        <!--<cylinder radius="0.0865" length="0.05234"/>-->
-        <mesh filename="file:$(find kridtbot)/meshes/wheel_assem.STL" scale="0.001 0.001 0.001"/>
-      </geometry>
-      <material name="orange"/>
-    </visual>
-    <collision>
-      <origin xyz="-0.085 0.085 0.035" rpy="1.57 0 0"/>
-      <geometry>
-        <mesh filename="file:$(find kridtbot)/meshes/wheel_assem.STL" scale="0.001 0.001 0.001"/>
-      </geometry>
-      <material name="mesh_color"/>
-    </collision>
-    <inertial>
-      <mass value="1.01100"/>
-      <inertia ixx="5844491.97e-9" ixy="-376.28e-9" ixz="-3671.08e-9" iyy="5842839.83e-9" iyz="-796.72e-9" izz="3646247.90e-9"/>
-    </inertial>
-  </link>
-  <gazebo reference="left_front_rev_link">
-    <material>Gazebo/Orange</material>
-    <mu1 value="3"/>
-    <mu2 value="3"/>
-    <slip1 value="1"/>
-    <slip2 value="1"/>
-    <kp>1000000.0</kp>
-    <kd>1.0</kd>
-  </gazebo>
   <!-- _____________ 2. RIGHT DIFF LINK____________-->
   <joint name="right_diff" type="fixed">
@@ -374,5 +300,5 @@
   </link>
   <gazebo reference="right_rear_lin_link">
-    <material>Gazebo/Black</material>
+    <material>Gazebo/Red</material>
   </gazebo>
    <!-- _____________Right REAR motor ____________-->
@@ -403,41 +329,5 @@
   </link>
   <!-- _____________RIGHT REAR wheel ____________-->
-  <joint name="right_rear_wheel" type="continuous">
-    <origin xyz="0 0 0" rpy="0 0 0"/>
-    <axis xyz="0 0 1"/>
-    <parent link="right_rear_motor_link"/>
-    <child link="right_rear_rev_link"/>
-    <dynamics damping="0.7" friction="1"/>
-  </joint>
-  <link name="right_rear_rev_link">
-    <visual>
-       <origin xyz="-0.085 0.085 0.035" rpy="1.57 0 0"/>
-      <geometry>
-        <!-- <cylinder radius="0.0865" length="0.05234"/> -->
-        <mesh filename="file:$(find kridtbot)/meshes/wheel_assem.STL" scale="0.001 0.001 0.001"/>
-      </geometry>
-      <material name="orange"/>
-    </visual>
-    <collision>
-       <origin xyz="-0.085 0.085 0.035" rpy="1.57 0 0"/>
-      <geometry>
-        <mesh filename="file:$(find kridtbot)/meshes/wheel_assem.STL" scale="0.001 0.001 0.001"/>
-      </geometry>
-      <material name="mesh_color"/>
-    </collision>
-    <inertial>
-      <mass value="1.01100"/>
-      <inertia ixx="5844491.97e-9" ixy="-376.28e-9" ixz="-3671.08e-9" iyy="5842839.83e-9" iyz="-796.72e-9" izz="3646247.90e-9"/>
-    </inertial>
-  </link>
-  <gazebo reference="right_rear_rev_link">
-    <material>Gazebo/Orange</material>
-    <mu1 value="3"/>
-    <mu2 value="3"/>
-    <slip1 value="1"/>
-    <slip2 value="1"/>
-    <kp>1000000.0</kp>
-    <kd>1.0</kd>
-  </gazebo>
+  <!-- See other page -->
   <!-- _____________RIGHT FRONT LINEAR actuator ____________-->
   <joint name="right_front_linear" type="prismatic">
@@ -469,5 +359,5 @@
   </link>
   <gazebo reference="right_front_lin_link">
-    <material>Gazebo/Black</material>
+    <material>Gazebo/Red</material>
   </gazebo>
     <!-- _____________Right front motor ____________-->
@@ -497,42 +387,4 @@
     </inertial>
   </link>
-  <!-- _____________RIGHT FRONT wheel ____________-->
-  <joint name="right_front_wheel" type="continuous">
-    <origin xyz="0.0 0 0" rpy="0 0 0"/>
-    <axis xyz="0 0 1"/>
-    <parent link="right_front_motor_link"/>
-    <child link="right_front_rev_link"/>
-    <dynamics damping="0.7" friction="1"/>
-  </joint>
-  <link name="right_front_rev_link">
-    <visual>
-      <origin xyz="-0.085 0.085 0.035" rpy="1.57 0 0"/>
-      <geometry>
-        <!-- <cylinder radius="0.0865" length="0.05234"/> -->
-        <mesh filename="file:$(find kridtbot)/meshes/wheel_assem.STL" scale="0.001 0.001 0.001"/>
-      </geometry>
-      <material name="orange"/>
-    </visual>
-    <collision>
-      <origin xyz="-0.085 0.085 0.035" rpy="1.57 0 0"/>
-      <geometry>
-        <mesh filename="file:$(find kridtbot)/meshes/wheel_assem.STL" scale="0.001 0.001 0.001"/>
-      </geometry>
-      <material name="mesh_color"/>
-    </collision>
-    <inertial>
-      <mass value="1.01100"/>
-      <inertia ixx="5844491.97e-9" ixy="-376.28e-9" ixz="-3671.08e-9" iyy="5842839.83e-9" iyz="-796.72e-9" izz="3646247.90e-9"/>
-    </inertial>
-  </link>
-  <gazebo reference="right_front_rev_link">
-    <material>Gazebo/Orange</material>
-    <mu1 value="3"/>
-    <mu2 value="3"/>
-    <slip1 value="1"/>
-    <slip2 value="1"/>
-    <kp>1000000.0</kp>
-    <kd>1.0</kd>
-  </gazebo>
 <!-- _____________ 3. CENTER DIFF LINK____________-->
   <joint name="center_diff" type="fixed">
@@ -567,4 +419,3 @@
     <mu2 value="1"/>
   </gazebo>
-  <!--   Differential gear -->
 </robot>

File: description/ros2_control_gz.xacro (robot description, xacro)
@@ -51,5 +51,5 @@
             <state_interface name="position"/>
             <state_interface name="velocity"/>
-            <state_interface name="effort"/>
+            <statelocalization_interface name="effort"/>
         </joint>
         <joint name="left_front_linear">
