Commit message: d

File: description/robot_core.xacro (robot description, xacro)
@@ -85,5 +85,5 @@
   </gazebo>
   <!-- _____________ 1. LEFT DIFF LINK ____________-->
-  <joint name="left_diff" type="fixed">
+  <joint name="left_diff" type="continuous">
     <origin xyz="0 0 -0.28" rpy="-3.1416 0 -3.1416"/>
     <axis xyz="0 0 1"/>
@@ -259,5 +259,5 @@
   </gazebo>
   <!-- _____________ 2. RIGHT DIFF LINK____________-->
-  <joint name="right_diff" type="fixed">
+  <joint name="right_diff" type="continuous">
     <origin xyz="0 0 0.28" rpy="0 0 0"/>
     <axis xyz="0 0 1"/>
@@ -428,5 +428,5 @@
   </gazebo>
 <!-- _____________ 3. CENTER DIFF LINK____________-->
-  <joint name="center_diff" type="fixed">
+  <joint name="center_diff" type="continuous">
     <origin xyz="0.0 0.05 0" rpy="1.57079632679 0 0"/> <!-- Adjusted orientation -->
     <axis xyz="0 0 1"/>  <!-- Rotates along X-axis -->

File: description/ros2_control_gz.xacro (robot description, xacro)
@@ -62,5 +62,5 @@
         </joint>
         <!-- IMU sensor-->
-        <sensor name="imu_sensor">
+        <sensor name="imu">
             <param name="frame_id">imu_link</param>
             <state_interface name="orientation.x"/>

Commit message: gazebo fix

File: description/robot_core.xacro (robot description, xacro)
@@ -85,5 +85,5 @@
   </gazebo>
   <!-- _____________ 1. LEFT DIFF LINK ____________-->
-  <joint name="left_diff" type="continuous">
+  <joint name="left_diff" type="fixed">
     <origin xyz="0 0 -0.28" rpy="-3.1416 0 -3.1416"/>
     <axis xyz="0 0 1"/>
@@ -259,5 +259,5 @@
   </gazebo>
   <!-- _____________ 2. RIGHT DIFF LINK____________-->
-  <joint name="right_diff" type="continuous">
+  <joint name="right_diff" type="fixed">
     <origin xyz="0 0 0.28" rpy="0 0 0"/>
     <axis xyz="0 0 1"/>
@@ -428,5 +428,5 @@
   </gazebo>
 <!-- _____________ 3. CENTER DIFF LINK____________-->
-  <joint name="center_diff" type="continuous">
+  <joint name="center_diff" type="fixed">
     <origin xyz="0.0 0.05 0" rpy="1.57079632679 0 0"/> <!-- Adjusted orientation -->
     <axis xyz="0 0 1"/>  <!-- Rotates along X-axis -->

Commit message: Changed path in URDF for meshes

File: description/robot_core.xacro (robot description, xacro)
@@ -32,5 +32,5 @@
       <origin xyz="0 0 0" rpy="0 0 0"/>
       <geometry>
-        <mesh filename="package://kridtbot/meshes/base_link.STL"/>
+        <mesh filename="file:$(find kridtbot)/meshes/base_link.STL"/>
       </geometry>
       <material name="orange"/>
@@ -39,5 +39,5 @@
       <origin xyz="0 0 0" rpy="0 0 0"/>
       <geometry>
-        <mesh filename="package://kridtbot/meshes/base_link.STL"/>
+        <mesh filename="file:$(find kridtbot)/meshes/base_link.STL"/>
       </geometry>
       <material name="mesh_color"/>
@@ -63,12 +63,12 @@
       <origin xyz="0 0 0" rpy="0 0 0"/>
       <geometry>
-        <mesh filename="package://kridtbot/meshes/diff_link.STL"/>
-      </geometry>
-      <material name="black"/>
-    </visual>
-    <collision>
-      <origin xyz="0 0 0" rpy="0 0 0"/>
-      <geometry>
-        <mesh filename="package://kridtbot/meshes/diff_link.STL"/>
+        <mesh filename="file:$(find kridtbot)/meshes/diff_link.STL"/>
+      </geometry>
+      <material name="black"/>
+    </visual>
+    <collision>
+      <origin xyz="0 0 0" rpy="0 0 0"/>
+      <geometry>
+        <mesh filename="file:$(find kridtbot)/meshes/diff_link.STL"/>
       </geometry>
       <material name="mesh_color"/>
@@ -103,12 +103,12 @@
       <origin xyz="0 0 0" rpy="0 0 0"/>
       <geometry>
-        <mesh filename="package://kridtbot/meshes/left_diff_link.STL"/>
-      </geometry>
-      <material name="black"/>
-    </visual>
-    <collision>
-      <origin xyz="0 0 0" rpy="0 0 0"/>
-      <geometry>
-        <mesh filename="package://kridtbot/meshes/left_diff_link.STL"/>
+        <mesh filename="file:$(find kridtbot)/meshes/left_diff_link.STL"/>
+      </geometry>
+      <material name="black"/>
+    </visual>
+    <collision>
+      <origin xyz="0 0 0" rpy="0 0 0"/>
+      <geometry>
+        <mesh filename="file:$(find kridtbot)/meshes/left_diff_link.STL"/>
       </geometry>
       <material name="mesh_color"/>
@@ -136,12 +136,12 @@
       <origin xyz="0 0 0" rpy="0 0 0"/>
       <geometry>
-        <mesh filename="package://kridtbot/meshes/left_rear_lin_link.STL"/>
-      </geometry>
-      <material name="black"/>
-    </visual>
-    <collision>
-      <origin xyz="0 0 0" rpy="0 0 0"/>
-      <geometry>
-        <mesh filename="package://kridtbot/meshes/left_rear_lin_link.STL"/>
+        <mesh filename="file:$(find kridtbot)/meshes/left_rear_lin_link.STL"/>
+      </geometry>
+      <material name="black"/>
+    </visual>
+    <collision>
+      <origin xyz="0 0 0" rpy="0 0 0"/>
+      <geometry>
+        <mesh filename="file:$(find kridtbot)/meshes/left_rear_lin_link.STL"/>
       </geometry>
       <material name="mesh_color"/>
@@ -193,12 +193,12 @@
       <origin xyz="0 0 0" rpy="0 0 0"/>
       <geometry>
-        <mesh filename="package://kridtbot/meshes/front_left_lin_link.STL"/>
-      </geometry>
-      <material name="black"/>
-    </visual>
-    <collision>
-      <origin xyz="0 0 0" rpy="0 0 0"/>
-      <geometry>
-        <mesh filename="package://kridtbot/meshes/front_left_lin_link.STL"/>
+        <mesh filename="file:$(find kridtbot)/meshes/front_left_lin_link.STL"/>
+      </geometry>
+      <material name="black"/>
+    </visual>
+    <collision>
+      <origin xyz="0 0 0" rpy="0 0 0"/>
+      <geometry>
+        <mesh filename="file:$(find kridtbot)/meshes/front_left_lin_link.STL"/>
       </geometry>
       <material name="mesh_color"/>
@@ -250,12 +250,12 @@
       <origin xyz="0 0 0" rpy="0 0 0"/>
       <geometry>
-        <mesh filename="package://kridtbot/meshes/rigth_diff_link.STL"/>
-      </geometry>
-      <material name="black"/>
-    </visual>
-    <collision>
-      <origin xyz="0 0 0" rpy="0 0 0"/>
-      <geometry>
-        <mesh filename="package://kridtbot/meshes/rigth_diff_link.STL"/>
+        <mesh filename="file:$(find kridtbot)/meshes/rigth_diff_link.STL"/>
+      </geometry>
+      <material name="black"/>
+    </visual>
+    <collision>
+      <origin xyz="0 0 0" rpy="0 0 0"/>
+      <geometry>
+        <mesh filename="file:$(find kridtbot)/meshes/rigth_diff_link.STL"/>
       </geometry>
       <material name="mesh_color"/>
@@ -283,12 +283,12 @@
       <origin xyz="0 0 0" rpy="0 0 0"/>
       <geometry>
-        <mesh filename="package://kridtbot/meshes/right_rear_lin_link.STL"/>
-      </geometry>
-      <material name="black"/>
-    </visual>
-    <collision>
-      <origin xyz="0 0 0" rpy="0 0 0"/>
-      <geometry>
-        <mesh filename="package://kridtbot/meshes/right_rear_lin_link.STL"/>
+        <mesh filename="file:$(find kridtbot)/meshes/right_rear_lin_link.STL"/>
+      </geometry>
+      <material name="black"/>
+    </visual>
+    <collision>
+      <origin xyz="0 0 0" rpy="0 0 0"/>
+      <geometry>
+        <mesh filename="file:$(find kridtbot)/meshes/right_rear_lin_link.STL"/>
       </geometry>
       <material name="mesh_color"/>
@@ -342,12 +342,12 @@
       <origin xyz="0 0 0" rpy="0 0 0"/>
       <geometry>
-        <mesh filename="package://kridtbot/meshes/right_front_lin_link.STL"/>
-      </geometry>
-      <material name="black"/>
-    </visual>
-    <collision>
-      <origin xyz="0 0 0" rpy="0 0 0"/>
-      <geometry>
-        <mesh filename="package://kridtbot/meshes/right_front_lin_link.STL"/>
+        <mesh filename="file:$(find kridtbot)/meshes/right_front_lin_link.STL"/>
+      </geometry>
+      <material name="black"/>
+    </visual>
+    <collision>
+      <origin xyz="0 0 0" rpy="0 0 0"/>
+      <geometry>
+        <mesh filename="file:$(find kridtbot)/meshes/right_front_lin_link.STL"/>
       </geometry>
       <material name="mesh_color"/>
