Commit message: Add real robot implementation

File: description/lidar.xacro (robot description, xacro)
@@ -47,9 +47,9 @@
         <parent link="lidar_stand_link"/>
         <child link="lidar_link"/>
-        <origin xyz="-0.002 -0.135 -0.185" rpy="0 0 0"/>
+        <origin xyz="-0.002 -0.135 -0.185" rpy="0 0 -1.57"/>
     </joint>
     <link name="lidar_link">
         <visual>
-            <origin xyz="0 0 0" rpy="1.57 0 1.57"/>
+            <origin xyz="0 0 0" rpy="1.57 0.0 3.14"/>
             <geometry>
                 <mesh filename="file:$(find kridtbot)/meshes/mid-360-asm copy.STL" scale="0.001 0.001 0.001"/>
@@ -73,5 +73,5 @@
                 <scan>
                     <horizontal>
-                        <samples>720</samples>
+                        <samples>360</samples>
                         <resolution>1</resolution>
                         <min_angle>0</min_angle>
@@ -87,5 +87,5 @@
                 <range>
                     <min>0.1</min>
-                    <max>70.0</max>
+                    <max>200.0</max>
                     <resolution>0.002</resolution>
                 </range>
@@ -93,5 +93,5 @@
                     <type>gaussian</type>
                     <mean>0.0</mean>
-                    <stddev>0.0001</stddev>
+                    <stddev>0.01</stddev>
                 </noise>
             </lidar>

File: description/robot.urdf.xacro (robot description, xacro)
@@ -24,5 +24,4 @@
         <xacro:include filename="ros2_control_myactuator.xacro" />
         <xacro:include filename="ros2_control_odrive.xacro" />
-        <xacro:include filename="ros2_control_imu.xacro" />
     </xacro:unless>
 </robot>

File: description/robot_core.xacro (robot description, xacro)
@@ -32,5 +32,5 @@
       <origin xyz="0 0 0" rpy="0 0 0"/>
       <geometry>
-        <mesh filename="file:$(find kridtbot)/meshes/base_link.STL"/>
+        <mesh filename="package://kridtbot/meshes/base_link.STL"/>
       </geometry>
       <material name="orange"/>
@@ -39,5 +39,5 @@
       <origin xyz="0 0 0" rpy="0 0 0"/>
       <geometry>
-        <mesh filename="file:$(find kridtbot)/meshes/base_link.STL"/>
+        <mesh filename="package://kridtbot/meshes/base_link.STL"/>
       </geometry>
       <material name="mesh_color"/>
@@ -63,12 +63,12 @@
       <origin xyz="0 0 0" rpy="0 0 0"/>
       <geometry>
-        <mesh filename="file:$(find kridtbot)/meshes/diff_link.STL"/>
-      </geometry>
-      <material name="black"/>
-    </visual>
-    <collision>
-      <origin xyz="0 0 0" rpy="0 0 0"/>
-      <geometry>
-        <mesh filename="file:$(find kridtbot)/meshes/diff_link.STL"/>
+        <mesh filename="package://kridtbot/meshes/diff_link.STL"/>
+      </geometry>
+      <material name="black"/>
+    </visual>
+    <collision>
+      <origin xyz="0 0 0" rpy="0 0 0"/>
+      <geometry>
+        <mesh filename="package://kridtbot/meshes/diff_link.STL"/>
       </geometry>
       <material name="mesh_color"/>
@@ -103,12 +103,12 @@
       <origin xyz="0 0 0" rpy="0 0 0"/>
       <geometry>
-        <mesh filename="file:$(find kridtbot)/meshes/left_diff_link.STL"/>
-      </geometry>
-      <material name="black"/>
-    </visual>
-    <collision>
-      <origin xyz="0 0 0" rpy="0 0 0"/>
-      <geometry>
-        <mesh filename="file:$(find kridtbot)/meshes/left_diff_link.STL"/>
+        <mesh filename="package://kridtbot/meshes/left_diff_link.STL"/>
+      </geometry>
+      <material name="black"/>
+    </visual>
+    <collision>
+      <origin xyz="0 0 0" rpy="0 0 0"/>
+      <geometry>
+        <mesh filename="package://kridtbot/meshes/left_diff_link.STL"/>
       </geometry>
       <material name="mesh_color"/>
@@ -136,12 +136,12 @@
       <origin xyz="0 0 0" rpy="0 0 0"/>
       <geometry>
-        <mesh filename="file:$(find kridtbot)/meshes/left_rear_lin_link.STL"/>
-      </geometry>
-      <material name="black"/>
-    </visual>
-    <collision>
-      <origin xyz="0 0 0" rpy="0 0 0"/>
-      <geometry>
-        <mesh filename="file:$(find kridtbot)/meshes/left_rear_lin_link.STL"/>
+        <mesh filename="package://kridtbot/meshes/left_rear_lin_link.STL"/>
+      </geometry>
+      <material name="black"/>
+    </visual>
+    <collision>
+      <origin xyz="0 0 0" rpy="0 0 0"/>
+      <geometry>
+        <mesh filename="package://kridtbot/meshes/left_rear_lin_link.STL"/>
       </geometry>
       <material name="mesh_color"/>
@@ -193,12 +193,12 @@
       <origin xyz="0 0 0" rpy="0 0 0"/>
       <geometry>
-        <mesh filename="file:$(find kridtbot)/meshes/front_left_lin_link.STL"/>
-      </geometry>
-      <material name="black"/>
-    </visual>
-    <collision>
-      <origin xyz="0 0 0" rpy="0 0 0"/>
-      <geometry>
-        <mesh filename="file:$(find kridtbot)/meshes/front_left_lin_link.STL"/>
+        <mesh filename="package://kridtbot/meshes/front_left_lin_link.STL"/>
+      </geometry>
+      <material name="black"/>
+    </visual>
+    <collision>
+      <origin xyz="0 0 0" rpy="0 0 0"/>
+      <geometry>
+        <mesh filename="package://kridtbot/meshes/front_left_lin_link.STL"/>
       </geometry>
       <material name="mesh_color"/>
@@ -250,12 +250,12 @@
       <origin xyz="0 0 0" rpy="0 0 0"/>
       <geometry>
-        <mesh filename="file:$(find kridtbot)/meshes/rigth_diff_link.STL"/>
-      </geometry>
-      <material name="black"/>
-    </visual>
-    <collision>
-      <origin xyz="0 0 0" rpy="0 0 0"/>
-      <geometry>
-        <mesh filename="file:$(find kridtbot)/meshes/rigth_diff_link.STL"/>
+        <mesh filename="package://kridtbot/meshes/rigth_diff_link.STL"/>
+      </geometry>
+      <material name="black"/>
+    </visual>
+    <collision>
+      <origin xyz="0 0 0" rpy="0 0 0"/>
+      <geometry>
+        <mesh filename="package://kridtbot/meshes/rigth_diff_link.STL"/>
       </geometry>
       <material name="mesh_color"/>
@@ -283,12 +283,12 @@
       <origin xyz="0 0 0" rpy="0 0 0"/>
       <geometry>
-        <mesh filename="file:$(find kridtbot)/meshes/right_rear_lin_link.STL"/>
-      </geometry>
-      <material name="black"/>
-    </visual>
-    <collision>
-      <origin xyz="0 0 0" rpy="0 0 0"/>
-      <geometry>
-        <mesh filename="file:$(find kridtbot)/meshes/right_rear_lin_link.STL"/>
+        <mesh filename="package://kridtbot/meshes/right_rear_lin_link.STL"/>
+      </geometry>
+      <material name="black"/>
+    </visual>
+    <collision>
+      <origin xyz="0 0 0" rpy="0 0 0"/>
+      <geometry>
+        <mesh filename="package://kridtbot/meshes/right_rear_lin_link.STL"/>
       </geometry>
       <material name="mesh_color"/>
@@ -342,12 +342,12 @@
       <origin xyz="0 0 0" rpy="0 0 0"/>
       <geometry>
-        <mesh filename="file:$(find kridtbot)/meshes/right_front_lin_link.STL"/>
-      </geometry>
-      <material name="black"/>
-    </visual>
-    <collision>
-      <origin xyz="0 0 0" rpy="0 0 0"/>
-      <geometry>
-        <mesh filename="file:$(find kridtbot)/meshes/right_front_lin_link.STL"/>
+        <mesh filename="package://kridtbot/meshes/right_front_lin_link.STL"/>
+      </geometry>
+      <material name="black"/>
+    </visual>
+    <collision>
+      <origin xyz="0 0 0" rpy="0 0 0"/>
+      <geometry>
+        <mesh filename="package://kridtbot/meshes/right_front_lin_link.STL"/>
       </geometry>
       <material name="mesh_color"/>
