Commit message: Code for physical robot

File: description/lidar.xacro (robot description, xacro)
@@ -1,16 +1,55 @@
 <?xml version="1.0"?>
 <robot xmlns:xacro="http://www.ros.org/wiki/xacro">
-    <!-- Fix Lidar Message type -->
-    <!-- Fix vertical sampling-->
-    <!-- Lidar Joint -->
-    <joint name="lidar_joint" type="fixed">
+    <!-- Lidar Base -->
+    <joint name="lidar_base_joint" type="fixed">
         <parent link="chassis_link"/>
-        <child link="lidar_link"/>
+        <child link="lidar_base_link"/>
         <origin xyz="0 0 -0.23" rpy="0 0 0"/>
     </joint>
-    <!-- Lidar Link -->
+    <link name="lidar_base_link">
+        <visual>
+            <origin xyz="-0.085 -0.2 -0.11" rpy="1.57 0 1.57"/>
+            <geometry>
+                <mesh filename="file:$(find kridtbot)/meshes/lidar_stand_base.STL" scale="0.001 0.001 0.001"/>
+            </geometry>
+            <material name="orange"/>
+        </visual>
+        <collision>
+            <origin xyz="-0.085 -0.2 -0.11" rpy="1.57 0 1.57"/>
+            <geometry>
+                <mesh filename="file:$(find kridtbot)/meshes/lidar_stand_base.STL" scale="0.001 0.001 0.001"/>
+            </geometry>
+        </collision>
+    </link>
+    <!-- Lidar Stand -->
+    <joint name="lidar_stand_joint" type="fixed">
+        <parent link="lidar_base_link"/>
+        <child link="lidar_stand_link"/>
+        <origin xyz="0 0 0" rpy="0 0 0"/>
+    </joint>
+    <link name="lidar_stand_link">
+        <visual>
+            <origin xyz="0.08 -0.2 0" rpy="-1.57 0 1.57"/>
+            <geometry>
+                <mesh filename="file:$(find kridtbot)/meshes/lidar_stand_top.STL" scale="0.001 0.001 0.001"/>
+            </geometry>
+            <material name="orange"/>
+        </visual>
+        <collision>
+            <origin xyz="0.08 -0.2 0" rpy="-1.57 0 1.57"/>
+            <geometry>
+                <mesh filename="file:$(find kridtbot)/meshes/lidar_stand_top.STL" scale="0.001 0.001 0.001"/>
+            </geometry>
+        </collision>
+    </link>
+    <!-- Lidar -->
+    <joint name="lidar_joint" type="fixed">
+        <parent link="lidar_stand_link"/>
+        <child link="lidar_link"/>
+        <origin xyz="-0.002 -0.135 -0.185" rpy="0 0 0"/>
+    </joint>
     <link name="lidar_link">
         <visual>
-            <origin xyz="0 0 0" rpy="-1.578 0 0"/>
+            <origin xyz="0 0 0" rpy="1.57 0 1.57"/>
             <geometry>
                 <mesh filename="file:$(find kridtbot)/meshes/mid-360-asm copy.STL" scale="0.001 0.001 0.001"/>
@@ -19,5 +58,5 @@
         </visual>
         <collision>
-            <origin xyz="0 0 0" rpy="-1.578 0 0"/>
+            <origin xyz="0 0 0" rpy="0 0 0"/>
             <geometry>
                 <mesh filename="file:$(find kridtbot)/meshes/mid-360-asm copy.STL" scale="0.001 0.001 0.001"/>
@@ -25,44 +64,35 @@
         </collision>
     </link>
-    <!-- FOV -->
-    <link name="lidar_optical_link">
-        <visual>
-            <geometry>
-                <mesh filename="file:$(find kridtbot)/meshes/mid-360-fov-asm.STL" scale="0.001 0.001 0.001"/>
-            </geometry>
-            <material name="blue opaque"/>
-        </visual>
-    </link>
-    <joint name="lidar_optical_joint" type="fixed">
-        <parent link="lidar_link"/>
-        <child link="lidar_optical_link"/>
-        <origin xyz="0 0 -0.02" rpy="-1.578 0 0"/>
-    </joint>
     <!-- Gazebo Sensor Definition -->
     <gazebo reference="lidar_link">
         <sensor type="gpu_lidar" name="lidar_sensor">
-            <visualize>false</visualize>  <!-- Visualization causes crashes, disable if needed -->
-            <pose>0 0 0 0 0 0</pose>
-            <update_rate>10</update_rate>  <!-- 10 Hz scan update -->
+            <visualize>true</visualize>
+            <pose>0 0 0 0 0 0</pose> <!-- 180 deg flip -->
+            <update_rate>100</update_rate>
             <lidar>
-            <!-- Information from Livox specs -->
                 <scan>
                     <horizontal>
-                        <samples>360</samples>  <!-- 360 points per rotation -->
-                        <!--<resolution>1</resolution> -->
-                        <min_angle>-3.14</min_angle>
-                        <max_angle>3.14</max_angle>
+                        <samples>360</samples>
+                        <resolution>1</resolution>
+                        <min_angle>0</min_angle>
+                        <max_angle>6.283185</max_angle> <!-- 360 deg -->
                     </horizontal>
                     <vertical>
-                        <samples>10</samples>  <!-- 1 vertical scan -->
-                        <min_angle>0</min_angle>
-                        <max_angle>-1</max_angle>
+                        <samples>100</samples>
+                        <resolution>1</resolution>
+                        <min_angle>-0.122</min_angle> <!-- -7.22 deg -->
+                        <max_angle>0.9</max_angle>  <!-- 55.22 deg seems to be to much-->
                     </vertical>
                 </scan>
                 <range>
-                    <min>0.1</min>  <!-- 10 cm min detection -->
-                    <max>12</max>  <!-- 70 m max detection -->
-                    <!--<resolution>0.02</resolution> -->  <!-- 2 cm precision -->
+                    <min>0.1</min>
+                    <max>200.0</max>
+                    <resolution>0.002</resolution>
                 </range>
+                <noise>
+                    <type>gaussian</type>
+                    <mean>0.0</mean>
+                    <stddev>0.01</stddev>
+                </noise>
             </lidar>
             <topic>lidar/points</topic>

File: description/robot.urdf.xacro (robot description, xacro)
@@ -14,7 +14,6 @@
     </xacro:if>
     <xacro:unless value="$(arg use_sim_system)">
-        <xacro:include filename="ros2_control_myactuator.xacro" />
-        <xacro:include filename="ros2_control_odrive.xacro" />
-        <xacro:include filename="ros2_control_imu.xacro" />
+        <xacro:include filename="ros2_control_myactuator.xacro"/>
+        <!--  <xacro:include filename="ros2_control_odrive.xacro" />-->
     </xacro:unless>
 </robot>

File: description/robot_core.xacro (robot description, xacro)
@@ -32,5 +32,5 @@
       <origin xyz="0 0 0" rpy="0 0 0"/>
       <geometry>
-        <mesh filename="file:$(find kridtbot)/meshes/base_link.STL"/>
+        <mesh filename="package://kridtbot/meshes/base_link.STL"/>
       </geometry>
       <material name="orange"/>
@@ -39,5 +39,5 @@
       <origin xyz="0 0 0" rpy="0 0 0"/>
       <geometry>
-        <mesh filename="file:$(find kridtbot)/meshes/base_link.STL"/>
+        <mesh filename="package://kridtbot/meshes/base_link.STL"/>
       </geometry>
       <material name="mesh_color"/>
@@ -63,12 +63,12 @@
       <origin xyz="0 0 0" rpy="0 0 0"/>
       <geometry>
-        <mesh filename="file:$(find kridtbot)/meshes/diff_link.STL"/>
-      </geometry>
-      <material name="black"/>
-    </visual>
-    <collision>
-      <origin xyz="0 0 0" rpy="0 0 0"/>
-      <geometry>
-        <mesh filename="file:$(find kridtbot)/meshes/diff_link.STL"/>
+        <mesh filename="package://kridtbot/meshes/diff_link.STL"/>
+      </geometry>
+      <material name="black"/>
+    </visual>
+    <collision>
+      <origin xyz="0 0 0" rpy="0 0 0"/>
+      <geometry>
+        <mesh filename="package://kridtbot/meshes/diff_link.STL"/>
       </geometry>
       <material name="mesh_color"/>
@@ -103,12 +103,12 @@
       <origin xyz="0 0 0" rpy="0 0 0"/>
       <geometry>
-        <mesh filename="file:$(find kridtbot)/meshes/left_diff_link.STL"/>
-      </geometry>
-      <material name="black"/>
-    </visual>
-    <collision>
-      <origin xyz="0 0 0" rpy="0 0 0"/>
-      <geometry>
-        <mesh filename="file:$(find kridtbot)/meshes/left_diff_link.STL"/>
+        <mesh filename="package://kridtbot/meshes/left_diff_link.STL"/>
+      </geometry>
+      <material name="black"/>
+    </visual>
+    <collision>
+      <origin xyz="0 0 0" rpy="0 0 0"/>
+      <geometry>
+        <mesh filename="package://kridtbot/meshes/left_diff_link.STL"/>
       </geometry>
       <material name="mesh_color"/>
@@ -125,5 +125,5 @@
   </gazebo>
   <!-- _____________LEFT REAR LINEAR ACtuator____________-->
-  <joint name="left_rear_linear" type="prismatic">
+  <joint name="left_rear_linear" type="fixed">
     <limit effort="1000.0" lower="0" upper="0.13" velocity="0.5"/>
     <origin xyz="-0.216 -0.0010724 0" rpy="-1.5708 0 0.0049647"/>
@@ -136,12 +136,12 @@
       <origin xyz="0 0 0" rpy="0 0 0"/>
       <geometry>
-        <mesh filename="file:$(find kridtbot)/meshes/left_rear_lin_link.STL"/>
-      </geometry>
-      <material name="black"/>
-    </visual>
-    <collision>
-      <origin xyz="0 0 0" rpy="0 0 0"/>
-      <geometry>
-        <mesh filename="file:$(find kridtbot)/meshes/left_rear_lin_link.STL"/>
+        <mesh filename="package://kridtbot/meshes/left_rear_lin_link.STL"/>
+      </geometry>
+      <material name="black"/>
+    </visual>
+    <collision>
+      <origin xyz="0 0 0" rpy="0 0 0"/>
+      <geometry>
+        <mesh filename="package://kridtbot/meshes/left_rear_lin_link.STL"/>
       </geometry>
       <material name="mesh_color"/>
@@ -191,5 +191,5 @@
   </gazebo>
   <!-- _____________LEFT FRONT LINEAR actuator____________-->
-  <joint name="left_front_linear" type="prismatic">
+  <joint name="left_front_linear" type="fixed">
     <limit effort="1000.0" lower="0" upper="0.13" velocity="0.5"/>
     <origin xyz="0.216 0.0010724 0" rpy="-1.5708 0 0.0049647"/>
@@ -202,12 +202,12 @@
       <origin xyz="0 0 0" rpy="0 0 0"/>
       <geometry>
-        <mesh filename="file:$(find kridtbot)/meshes/front_left_lin_link.STL"/>
-      </geometry>
-      <material name="black"/>
-    </visual>
-    <collision>
-      <origin xyz="0 0 0" rpy="0 0 0"/>
-      <geometry>
-        <mesh filename="file:$(find kridtbot)/meshes/front_left_lin_link.STL"/>
+        <mesh filename="package://kridtbot/meshes/front_left_lin_link.STL"/>
+      </geometry>
+      <material name="black"/>
+    </visual>
+    <collision>
+      <origin xyz="0 0 0" rpy="0 0 0"/>
+      <geometry>
+        <mesh filename="package://kridtbot/meshes/front_left_lin_link.STL"/>
       </geometry>
       <material name="mesh_color"/>
@@ -270,12 +270,12 @@
       <origin xyz="0 0 0" rpy="0 0 0"/>
       <geometry>
-        <mesh filename="file:$(find kridtbot)/meshes/rigth_diff_link.STL"/>
-      </geometry>
-      <material name="black"/>
-    </visual>
-    <collision>
-      <origin xyz="0 0 0" rpy="0 0 0"/>
-      <geometry>
-        <mesh filename="file:$(find kridtbot)/meshes/rigth_diff_link.STL"/>
+        <mesh filename="package://kridtbot/meshes/rigth_diff_link.STL"/>
+      </geometry>
+      <material name="black"/>
+    </visual>
+    <collision>
+      <origin xyz="0 0 0" rpy="0 0 0"/>
+      <geometry>
+        <mesh filename="package://kridtbot/meshes/rigth_diff_link.STL"/>
       </geometry>
       <material name="mesh_color"/>
@@ -292,5 +292,5 @@
   </gazebo>
   <!-- _____________RIGHT REAR LINEAR actuator ____________-->
-  <joint name="right_rear_linear" type="prismatic">
+  <joint name="right_rear_linear" type="fixed">
     <limit effort="1000.0" lower="0" upper="0.13" velocity="0.5"/>
     <origin xyz="0.216 -0.0010724 0" rpy="-1.5708 0 0.0049647"/>
@@ -303,12 +303,12 @@
       <origin xyz="0 0 0" rpy="0 0 0"/>
       <geometry>
-        <mesh filename="file:$(find kridtbot)/meshes/right_rear_lin_link.STL"/>
-      </geometry>
-      <material name="black"/>
-    </visual>
-    <collision>
-      <origin xyz="0 0 0" rpy="0 0 0"/>
-      <geometry>
-        <mesh filename="file:$(find kridtbot)/meshes/right_rear_lin_link.STL"/>
+        <mesh filename="package://kridtbot/meshes/right_rear_lin_link.STL"/>
+      </geometry>
+      <material name="black"/>
+    </visual>
+    <collision>
+      <origin xyz="0 0 0" rpy="0 0 0"/>
+      <geometry>
+        <mesh filename="package://kridtbot/meshes/right_rear_lin_link.STL"/>
       </geometry>
       <material name="mesh_color"/>
@@ -360,5 +360,5 @@
   </gazebo>
   <!-- _____________RIGHT FRONT LINEAR actuator ____________-->
-  <joint name="right_front_linear" type="prismatic">
+  <joint name="right_front_linear" type="fixed">
     <limit effort="1000.0" lower="0" upper="0.13" velocity="0.5"/>
     <origin xyz="-0.216 0.0010724 0" rpy="-1.5708 0 0.0049647"/>
@@ -371,12 +371,12 @@
       <origin xyz="0 0 0" rpy="0 0 0"/>
       <geometry>
-        <mesh filename="file:$(find kridtbot)/meshes/right_front_lin_link.STL"/>
-      </geometry>
-      <material name="black"/>
-    </visual>
-    <collision>
-      <origin xyz="0 0 0" rpy="0 0 0"/>
-      <geometry>
-        <mesh filename="file:$(find kridtbot)/meshes/right_front_lin_link.STL"/>
+        <mesh filename="package://kridtbot/meshes/right_front_lin_link.STL"/>
+      </geometry>
+      <material name="black"/>
+    </visual>
+    <collision>
+      <origin xyz="0 0 0" rpy="0 0 0"/>
+      <geometry>
+        <mesh filename="package://kridtbot/meshes/right_front_lin_link.STL"/>
       </geometry>
       <material name="mesh_color"/>

File: description/ros2_control_myactuator.xacro (robot description, xacro)
@@ -1,16 +1,15 @@
 <?xml version="1.0"?>
 <robot xmlns:xacro="http://www.ros.org/wiki/xacro">
-    <!-- ROS2 Control plugin for Gazebo-->
-    <ros2_control name="myactuator_controller_right_rear_wheel" type="actuator">
+    <ros2_control name="myactuator_controller_right_front_wheel" type="actuator">
         <hardware>
             <plugin>myactuator_rmd_hardware/MyActuatorRmdHardwareInterface</plugin>
-            <param name="ifname">can1</param>
+            <param name="ifname">can2</param>
             <param name="actuator_id">5</param>
             <param name="torque_constant">2.023914969</param>
             <param name="velocity_alpha">0.1</param>
             <param name="effort_alpha">0.1</param>
-            <param name="cycle_time">1</param>
+            <param name="direction">1.0</param>
         </hardware>
-        <joint name="right_rear_wheel">
+        <joint name="right_front_wheel">
             <command_interface name="position"/>
             <command_interface name="velocity"/>
@@ -21,15 +20,15 @@
         </joint>
     </ros2_control>
-    <ros2_control name="myactuator_controller_right_front_wheel" type="actuator">
+    <ros2_control name="myactuator_controller_right_rear_wheel" type="actuator">
         <hardware>
             <plugin>myactuator_rmd_hardware/MyActuatorRmdHardwareInterface</plugin>
-            <param name="ifname">can2</param>
-            <param name="actuator_id">4</param>
+            <param name="ifname">can1</param>
+            <param name="actuator_id">7</param>
             <param name="torque_constant">2.023914969</param>
             <param name="velocity_alpha">0.1</param>
             <param name="effort_alpha">0.1</param>
-            <param name="cycle_time">1</param>
+            <param name="direction">1.0</param>
         </hardware>
-        <joint name="right_front_wheel">
+        <joint name="right_rear_wheel">
             <command_interface name="position"/>
             <command_interface name="velocity"/>
@@ -43,10 +42,10 @@
         <hardware>
             <plugin>myactuator_rmd_hardware/MyActuatorRmdHardwareInterface</plugin>
-            <param name="ifname">can3</param>
-            <param name="actuator_id">6</param>
+            <param name="ifname">can4</param>
+            <param name="actuator_id">4</param>
             <param name="torque_constant">2.023914969</param>
             <param name="velocity_alpha">0.1</param>
             <param name="effort_alpha">0.1</param>
-            <param name="cycle_time">1</param>
+            <param name="direction">-1.0</param>
         </hardware>
         <joint name="left_front_wheel">
@@ -62,10 +61,10 @@
         <hardware>
             <plugin>myactuator_rmd_hardware/MyActuatorRmdHardwareInterface</plugin>
-            <param name="ifname">can4</param>
-            <param name="actuator_id">7</param>
+            <param name="ifname">can3</param>
+            <param name="actuator_id">6</param>
             <param name="torque_constant">2.023914969</param>
             <param name="velocity_alpha">0.1</param>
             <param name="effort_alpha">0.1</param>
-            <param name="cycle_time">1</param>
+            <param name="direction">-1.0</param>
         </hardware>
         <joint name="left_rear_wheel">

File: description/ros2_control_odrive.xacro (robot description, xacro)
@@ -7,33 +7,9 @@
             <param name="can">can0</param>
         </hardware>
-        <joint name="right_rear_linear">
-            <param name="node_id">2</param>
-            <command_interface name="position">
-                <param name="min">-0.005</param>
-                <param name="max">0.10</param>
-            </command_interface>
-            <command_interface name="velocity"/>
-            <command_interface name="effort"/>
-            <state_interface name="position"/>
-            <state_interface name="velocity"/>
-            <state_interface name="effort"/>
-        </joint>
-        <joint name="right_front_linear">
-            <param name="node_id">3</param>
-            <command_interface name="position">
-                <param name="min">-0.005</param>
-                <param name="max">0.10</param>
-            </command_interface>
-            <command_interface name="velocity"/>
-            <command_interface name="effort"/>
-            <state_interface name="position"/>
-            <state_interface name="velocity"/>
-            <state_interface name="effort"/>
-        </joint>
         <joint name="left_rear_linear">
             <param name="node_id">1</param>
             <command_interface name="position">
                 <param name="min">-0.005</param>
-                <param name="max">0.10</param>
+                <param name="max">0.11</param>
             </command_interface>
             <command_interface name="velocity"/>
@@ -47,5 +23,31 @@
             <command_interface name="position">
                 <param name="min">-0.005</param>
-                <param name="max">0.10</param>
+                <param name="max">0.11</param>
+            </command_interface>
+            <command_interface name="velocity"/>
+            <command_interface name="effort"/>
+            <state_interface name="position"/>
+            <state_interface name="velocity"/>
+            <state_interface name="effort"/>
+        </joint>
+        <joint name="right_rear_linear">
+            <param name="node_id">2</param>
+            <command_interface name="position">
+                <param name="min">-0.005</param>
+                <param name="max">0.11</param>
+            </command_interface>
+            <command_interface name="velocity">
+                <param name="max">1.0</param>
+            </command_interface>
+            <command_interface name="effort"/>
+            <state_interface name="position"/>
+            <state_interface name="velocity"/>
+            <state_interface name="effort"/>
+        </joint>
+        <joint name="right_front_linear">
+            <param name="node_id">3</param>
+            <command_interface name="position">
+                <param name="min">-0.005</param>
+                <param name="max">0.11</param>
             </command_interface>
             <command_interface name="velocity"/>
